File: kicad_project/Relay.kicad_pcb (KiCad board)
At the start: 2 copper layers, 39.6 x 28.3 mm, 13 parts, among them J1 5018762640, J2 USB_C_Receptacle, J3 RJ45, K1 G6K-2P-Y_DC3, Q1 SO2222

Commit message: BOM and OSHW Logo
Other:
- board text added: "by loetkolben"
- board text removed: "loetkolben"

Commit message: added two more 12V vias
Routing:
- net +12V: vias 2 -> 4
Changed lines of the file:
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@@
   (segment (start 151.44 73.82) (end 150.18 73.82) (width 0.3) (layer "F.Cu") (net 12))
   (segment (start 150.18 73.82) (end 150.13 73.87) (width 0.25) (layer "F.Cu") (net 12))
+  (via (at 162.85 64.13) (size 0.8) (drill 0.4) (layers "F.Cu" "B.Cu") (net 12))
+  (via (at 161.815 65.165) (size 0.8) (drill 0.4) (layers "F.Cu" "B.Cu") (net 12))
   (via (at 163.52 62.71) (size 0.8) (drill 0.4) (layers "F.Cu" "B.Cu") (net 12))
   (via (at 160.79 66.19) (size 0.8) (drill 0.4) (layers "F.Cu" "B.Cu") (net 12))
@@
   (segment (start 150.13 76.27) (end 152.58 76.27) (width 0.5) (layer "B.Cu") (net 12))
   (segment (start 154.470489 74.379511) (end 154.470489 72.38913) (width 0.5) (layer "B.Cu") (net 12))
+  (segment (start 162.85 64.13) (end 161.815 65.165) (width 0.75) (layer "B.Cu") (net 12))
   (segment (start 152.58 76.27) (end 154.470489 74.379511) (width 0.5) (layer "B.Cu") (net 12))
   (segment (start 154.470489 72.38913) (end 155.06 71.799619) (width 0.5) (layer "B.Cu") (net 12))
-  (segment (start 163.52 63.46) (end 160.79 66.19) (width 0.75) (layer "B.Cu") (net 12))
+  (segment (start 163.52 63.46) (end 162.85 64.13) (width 0.75) (layer "B.Cu") (net 12))
   (segment (start 156.33 64.1975) (end 157.6 65.4675) (width 1) (layer "B.Cu") (net 12))
+  (segment (start 161.815 65.165) (end 160.79 66.19) (width 0.75) (layer "B.Cu") (net 12))
   (segment (start 163.52 62.71) (end 172.2675 62.71) (width 0.75) (layer "B.Cu") (net 12))
   (segment (start 157.6 65.4675) (end 160.0675 65.4675) (width 1) (layer "B.Cu") (net 12))

Commit message: thicker ignition line
Routing:
- net IGN: track 31.3 -> 35.0 mm, vias 1 -> 2
Changed lines of the file:
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@@
   (via (at 145.01 75.81) (size 0.8) (drill 0.4) (layers "F.Cu" "B.Cu") (free) (net 2))
   (via (at 144.98 73.98) (size 0.8) (drill 0.4) (layers "F.Cu" "B.Cu") (free) (net 2))
-  (segment (start 175.06 71.59) (end 175.18 71.71) (width 0.25) (layer "B.Cu") (net 2))
-  (segment (start 167.12546 70.83904) (end 172.85904 70.83904) (width 0.25) (layer "B.Cu") (net 2))
+  (segment (start 175.18 71.71) (end 175.18 77.5625) (width 0.25) (layer "B.Cu") (net 2))
+  (segment (start 167.0645 70.9) (end 172.071522 70.9) (width 0.25) (layer "B.Cu") (net 2))
   (segment (start 150.13 72.27) (end 149.64 71.78) (width 0.25) (layer "B.Cu") (net 2))
-  (segment (start 175.18 77.5625) (end 174.15 78.5925) (width 0.25) (layer "B.Cu") (net 2))
+  (segment (start 172.071522 70.9) (end 172.761522 71.59) (width 0.25) (layer "B.Cu") (net 2))
   (segment (start 149.64 71.05) (end 149.53 70.94) (width 0.25) (layer "B.Cu") (net 2))
   (segment (start 149.64 71.78) (end 149.64 71.05) (width 0.25) (layer "B.Cu") (net 2))
-  (segment (start 172.85904 70.83904) (end 173.61 71.59) (width 0.25) (layer "B.Cu") (net 2))
-  (segment (start 175.18 71.71) (end 175.18 77.5625) (width 0.25) (layer "B.Cu") (net 2))
-  (segment (start 165.9745 71.99) (end 167.12546 70.83904) (width 0.25) (layer "B.Cu") (net 2))
-  (segment (start 173.61 71.59) (end 175.06 71.59) (width 0.25) (layer "B.Cu") (net 2))
+  (segment (start 172.761522 71.59) (end 175.06 71.59) (width 0.25) (layer "B.Cu") (net 2))
+  (segment (start 165.9745 71.99) (end 167.0645 70.9) (width 0.25) (layer "B.Cu") (net 2))
+  (segment (start 175.06 71.59) (end 175.18 71.71) (width 0.25) (layer "B.Cu") (net 2))
+  (segment (start 175.18 77.5625) (end 174.15 78.5925) (width 0.25) (layer "B.Cu") (net 2))
   (segment (start 163.115 68.33) (end 161.145 68.33) (width 1) (layer "F.Cu") (net 3))
-  (segment (start 163.31 69.15) (end 163.115 68.955) (width 0.25) (layer "F.Cu") (net 3))
+  (segment (start 161.18 69.05) (end 161.145 69.015) (width 0.25) (layer "F.Cu") (net 3))
+  (segment (start 163.31 69.15) (end 163.21 69.05) (width 0.25) (layer "F.Cu") (net 3))
+  (segment (start 163.31 68.525) (end 163.115 68.33) (width 0.25) (layer "F.Cu") (net 3))
+  (segment (start 161.145 69.015) (end 161.145 68.33) (width 0.25) (layer "F.Cu") (net 3))
   (segment (start 163.31 70.8625) (end 163.41 70.9625) (width 0.25) (layer "F.Cu") (net 3))
-  (segment (start 163.115 68.955) (end 163.115 68.33) (width 0.25) (layer "F.Cu") (net 3))
-  (segment (start 163.31 69.15) (end 163.31 70.8625) (width 0.25) (layer "F.Cu") (net 3))
+  (segment (start 163.31 70.32) (end 163.31 70.8625) (width 0.25) (layer "F.Cu") (net 3))
+  (segment (start 163.21 69.05) (end 161.18 69.05) (width 0.4) (layer "F.Cu") (net 3))
+  (segment (start 163.31 69.15) (end 163.31 68.525) (width 0.25) (layer "F.Cu") (net 3))
   (via (at 163.31 69.15) (size 0.8) (drill 0.4) (layers "F.Cu" "B.Cu") (net 3))
-  (segment (start 172.8025 69.94) (end 174.15 68.5925) (width 0.25) (layer "B.Cu") (net 3))
-  (segment (start 175.16 55.6025) (end 175.16 67.5825) (width 0.25) (layer "B.Cu") (net 3))
-  (segment (start 163.31 69.15) (end 164.1 69.94) (width 0.25) (layer "B.Cu") (net 3))
-  (segment (start 164.1 69.94) (end 172.8025 69.94) (width 0.25) (layer "B.Cu") (net 3))
-  (segment (start 174.15 54.5925) (end 175.16 55.6025) (width 0.25) (layer "B.Cu") (net 3))
-  (segment (start 175.16 67.5825) (end 174.15 68.5925) (width 0.25) (layer "B.Cu") (net 3))
+  (via (at 163.31 70.32) (size 0.8) (drill 0.4) (layers "F.Cu" "B.Cu") (net 3))
+  (segment (start 172.8025 69.94) (end 174.15 68.5925) (width 0.4) (layer "B.Cu") (net 3))
+  (segment (start 175.16 55.6025) (end 175.16 67.5825) (width 0.4) (layer "B.Cu") (net 3))
+  (segment (start 163.945 69.785) (end 164.1 69.94) (width 0.4) (layer "B.Cu") (net 3))
+  (segment (start 164.1 69.94) (end 172.8025 69.94) (width 0.4) (layer "B.Cu") (net 3))
+  (segment (start 163.31 70.32) (end 163.845 69.785) (width 0.5) (layer "B.Cu") (net 3))
+  (segment (start 163.845 69.785) (end 163.945 69.785) (width 0.25) (layer "B.Cu") (net 3))
+  (segment (start 163.31 69.15) (end 163.31 70.32) (width 0.5) (layer "B.Cu") (net 3))
+  (segment (start 163.31 69.15) (end 163.945 69.785) (width 0.4) (layer "B.Cu") (net 3))
+  (segment (start 174.15 54.5925) (end 175.16 55.6025) (width 0.4) (layer "B.Cu") (net 3))
+  (segment (start 175.16 67.5825) (end 174.15 68.5925) (width 0.4) (layer "B.Cu") (net 3))
   (segment (start 174.15 56.5925) (end 176.15 56.5925) (width 0.25) (layer "F.Cu") (net 4))
   (segment (start 172.2 63.79) (end 171.015 62.605) (width 0.25) (layer "F.Cu") (net 4))
