File: kicad_project/Relay.kicad_sch (KiCad schematic)
At the start: 13 parts, among them J1 5018762640, J2 USB_C_Receptacle, J3 RJ45, K1 G6K-2P-Y_DC5, Q1 DDTC114ECA-7-F

Commit message: update usb-c and pcb
Parts:
- J2: footprint Connector_USB:USB_C_Receptacle_Amphenol_12401548E4-2A -> Relay:TYPE-C-31-M-04
Changed lines of the file:
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@@
       (effects (font (size 1.27 1.27)) (justify right))
     )
-    (property "Footprint" "Connector_USB:USB_C_Receptacle_Amphenol_12401548E4-2A" (id 2) (at 227.33 82.55 0)
+    (property "Footprint" "Relay:TYPE-C-31-M-04" (id 2) (at 227.33 82.55 0)
       (effects (font (size 1.27 1.27)) hide)
     )
@@
     )
     (path "/5abc6ae4-0eef-40a4-813f-08a489752b6e"
-      (reference "J2") (unit 1) (value "USB_C_Receptacle") (footprint "Connector_USB:USB_C_Receptacle_Amphenol_12401548E4-2A")
+      (reference "J2") (unit 1) (value "USB_C_Receptacle") (footprint "Relay:TYPE-C-31-M-04")
     )
     (path "/4e10830e-8b39-46a9-8dc1-85b40a1697bd"
